File: EA1176_TiGANBoard/EA1176_SOM.sch (KiCad schematic (older format))
At the start: 9 parts, among them J2 L829-1J1T-43, J4 Conn_ARM_JTAG_SWD_10, Q1 BSS138PW, Q2 BSS138PW, U1 iMXRT1176uCOM

Commit message: [fix] CADを更新 V1.0 beta
Parts:
- added D1: RB521S30T1G, Diode_SMD:D_SOD-523, symbol Device:D_Schottky_Small
- added D2: PESD5V0L5UV, Package_TO_SOT_SMD:SOT-666, symbol Power_Protection:PESD3V3L5UV
- added R10, R11, R12, R9: 50, Resistor_SMD:R_0402_1005Metric, symbol Device:R_Small
- added R13: 1k, Resistor_SMD:R_0402_1005Metric, symbol Device:R_Small
- added R8: 10k, Resistor_SMD:R_0402_1005Metric, symbol Device:R_Small
Connections:
- net PERI_3V3 is gone; now on net VDD_3V3: J2.16
- net GND: now also D2.2 (A), R13.2
- net JTAG_MOD: now also R13.1
- net JTAG_TCK: now also R9.1; no longer J4.4 (SWDCLK/TCK)
- net JTAG_TDI: now also R12.1; no longer J4.8 (NC/TDI)
- net JTAG_TDO: now also R11.1; no longer J4.6 (SWO/TDO)
- net JTAG_TMS: now also R10.1; no longer J4.2 (SWDIO/TMS)
- net JTAG_TRST: no longer J4.10 (~RESET~)
- net JTAG_VCC: now also R8.2
- net CAN1_EXT_TICK: now reaches U1.89 (GPIO_DISP_B2_11)
- net CAN1_TX: now reaches U1.93 (GPIO_DISP_B2_12)
- net CAN1_RX: now reaches U1.95 (GPIO_DISP_B2_13)
- net USER_SW: now reaches U1.142 (GPIO_SD_B2_02)
- net POR_B: now reaches U1.170 (POR_B)
- net POR_B: now also D1.2 (A)
- net ADC2_A6 renamed UART_TX
- net ADC2_B6 renamed UART_RX
- new net Conn_RST: D1.1 (K), D2.1 (K1), J4.10 (~RESET~), R8.1
- new net Conn_TCK: D2.5 (K4), J4.4 (SWDCLK/TCK), R9.2
- new net Conn_TDI: D2.3 (K2), J4.8 (NC/TDI), R12.2
- new net Conn_TDO: D2.6 (K5), J4.6 (SWO/TDO), R11.2
- new net Conn_TMS: D2.4 (K3), J4.2 (SWDIO/TMS), R10.2
- no-connect marks 185 -> 182
Other:
- note added: "ESD Protection"
- moved on the sheet: J4

Commit message: [fix]RJ45のうねうねを追加
Changed lines of the file:
@@
 Text HLabel 15000 5350 2    50   Output ~ 0
 UART_TX
+Text Label 10800 2500 0    50   ~ 0
+TRD1+
+Text Label 10800 2700 0    50   ~ 0
+TRD1-
+Text Label 10800 2900 0    50   ~ 0
+TRD2+
+Text Label 10800 3100 0    50   ~ 0
+TRD2-
+Text Label 10800 3300 0    50   ~ 0
+TRD3+
+Text Label 10800 3500 0    50   ~ 0
+TRD3-
+Text Label 10800 3700 0    50   ~ 0
+TRD4+
+Text Label 10800 3900 0    50   ~ 0
+TRD4-
 $EndSCHEMATC
