File: EA1176_TiGANBoard/EA1176_TiGANBoard.sch (KiCad schematic (older format))
At the start: 1 part, among them J1 Conn_01x04_Male

Commit message: [fix] CADを更新 V1.0 beta
Parts:
- removed J1: Conn_01x04_Male, Connector_PinHeader_2.54mm:PinHeader_1x04_P2.54mm_Vertical, symbol Connector:Conn_01x04_Male
- added C2: 0.1u, Capacitor_SMD:C_0402_1005Metric, symbol Device:C_Small
- added C3, C5: 0.1u, Capacitor_SMD:C_0402_1005Metric, symbol Device:C
- added C4: 1u, Capacitor_SMD:C_0402_1005Metric, symbol Device:C
- added D3: PESD5V0L5UV, Package_TO_SOT_SMD:SOT-666, symbol Power_Protection:PESD3V3L5UV
- added J1, J3: Conn_01x03, Connector_PinHeader_2.54mm:PinHeader_1x03_P2.54mm_Vertical, symbol Connector_Generic:Conn_01x03
- added J5: Conn_01x04, Connector_JST:JST_XH_B4B-XH-A_1x04_P2.50mm_Vertical, symbol Connector_Generic:Conn_01x04
- added J6: Conn_01x04, Connector_PinHeader_2.54mm:PinHeader_1x04_P2.54mm_Vertical, symbol Connector_Generic:Conn_01x04
- added R4: 10k, Resistor_SMD:R_0402_1005Metric, symbol Device:R_Small
- added R5: 100, Resistor_SMD:R_0402_1005Metric, symbol Device:R_Small
- added R6, R7: 60, Resistor_SMD:R_0402_1005Metric, symbol Device:R
- added SW1: SW_MEC_5E, Button_Switch_THT:SW_TH_Tactile_Omron_B3F-10xx, symbol Switch:SW_MEC_5E
- added TP1, TP2, TP3, TP4: TestPoint, Connector_PinHeader_2.54mm:PinHeader_1x01_P2.54mm_Vertical, symbol Connector:TestPoint
- added U3: TCAN332G, Package_TO_SOT_SMD:SOT-23-8, symbol Interface_CAN_LIN:TCAN332G
Connections:
- net ADC_U1: now also J3.2 (Pin_2)
- net ADC_U2: now also J1.2 (Pin_2)
- net GND: now also C2.2, C3.1, C4.1, C5.1, D3.2 (A), J1.3 (Pin_3), J3.3 (Pin_3), J5.1 (Pin_1), J5.4 (Pin_4), J6.4 (Pin_4), SW1.3 (K), SW1.4 (A), TP4.1, U3.2 (GND)
- net PWM_TRIG: now also D3.5 (K4), TP2.1
- net USER_GPIO: now also D3.4 (K3), TP3.1
- new net: C5.2, R6.2, R7.1
- new net +3V3: C3.2, C4.2, J1.1 (Pin_1), J3.1 (Pin_1), J6.1 (Pin_1), R4.2, TP1.1, U3.3 (VCC)
- new net CAN+: J5.3 (Pin_3), R6.1, U3.7 (CANH)
- new net CAN-: J5.2 (Pin_2), R7.2, U3.6 (CANL)
- new net CAN1_RX: U3.4 (RXD)
- new net CAN1_TX: U3.1 (TXD)
- new net UART_RX: D3.1 (K1), J6.2 (Pin_2)
- new net UART_TX: D3.3 (K2), J6.3 (Pin_3)
- new net USER_SW: R4.1, R5.2
- new net USER_SW_BTN: C2.1, D3.6 (K5), R5.1, SW1.1, SW1.2
Other:
- note added: "ESD Protection"
